Commit message: 修复BUG：fix(slam): 修复Cartographer建图时的崩溃与数据丢失问题
1.EKF时间戳校正：注释EKF节点提前0.1s的时间戳配置
2.Cartographer配置调优：降低lookup_transform_timeout_sec值、开启IMU数据融合，提升建图质量
3.修改URDF模型，将IMU位置修改到base_footprint中心,确保Cartographer可以正常建图与定位
因为EKF只需要IMU的角速度，而刚体的角速度与IMU位置无关，所以修改这个位置不影响EKF
Cartographer更重视IMU角速度，因为是2D Cartographer不是3D Cartographer，所以对IMU线速度的权重不如角速度，所以为了使用IMU数据，我们选择为了能用IMU数据，我们就干扰IMU角速度，最后效果还是有大大提升的

File: src/tianracer/tianracer_description/urdf/tianracer_compact.urdf.xacro (robot description, xacro)
@@ -63,7 +63,7 @@
   </link>
   <joint name="base_link_to_imu" type="fixed">
-    <parent link="${tf_prefix}base_link" />
+    <parent link="${tf_prefix}base_footprint" />
     <child link="${tf_prefix}imu_link" />
-    <origin xyz="0.22 0 0.1" rpy="0 0 0"/>
+    <origin xyz="0 0 0" rpy="0 0 0"/>
   </joint>
   <link
